Commit message: my changes

File: models/shadowhand.urdf (robot description, URDF)
Before this commit: robot shadowhand, 36 links, 35 joints
Links:
- removed link base_footprint
- removed link virtual_px_link
- removed link virtual_py_link
- removed link virtual_pz_link
- removed link virtual_rp_link
- removed link virtual_ry_link
- added link rh_forearm, mass 3.0; collision box size=0.07 0.07 0.07; collision mesh filename=package://sr_description/meshes/components/forearm/forearm_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 scale=0.001 0.001 0.001
- added link rh_manipulator
- added link rh_wrist, mass 0.1; collision box size=0.027 0.018 0.010; collision box size=0.027 0.018 0.010
- link rh_ffdistal: geometry collision mesh filename=package://sr_description/meshes/components/f_distal/pst/f_d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 scale=0.001 0.001 0.001; visual mesh filename=package://sr_description/meshes/components/f_distal/pst/f_d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 scale=0.001 0.001 0.001
- link rh_ffknuckle: geometry collision cylinder length=0.014 radius=0.007; visual mesh filename=package://sr_description/meshes/components/f_knuckle/f_knuc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 scale=0.001 0.001 0.001
- link rh_ffmiddle: geometry collision cylinder length=0.025 radius=0.007; collision sphere radius=0.007
- link rh_ffproximal: geometry collision cylinder length=0.040 radius=0.007; visual mesh filename=package://sr_description/meshes/components/f_proximal/f_pro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 scale=0.001 0.001 0.001
- link rh_lfdistal: geometry collision mesh filename=package://sr_description/meshes/components/f_distal/pst/f_d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 scale=0.001 0.001 0.001; visual mesh filename=package://sr_description/meshes/components/f_distal/pst/f_d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 scale=0.001 0.001 0.001
- link rh_lfknuckle: geometry collision cylinder length=0.014 radius=0.007; visual mesh filename=package://sr_description/meshes/components/f_knuckle/f_knuc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 scale=0.001 0.001 0.001
- link rh_lfmetacarpal: geometry collision box size=0.018 0.024 0.040; visual mesh filename=package://sr_description/meshes/components/lf_metacarpal/lf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 scale=0.001 0.001 0.001
- link rh_lfmiddle: geometry collision cylinder length=0.025 radius=0.007; collision sphere radius=0.007
- link rh_lfproximal: geometry collision cylinder length=0.040 radius=0.007; visual mesh filename=package://sr_description/meshes/components/f_proximal/f_pro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 scale=0.001 0.001 0.001
- link rh_mfdistal: geometry collision mesh filename=package://sr_description/meshes/components/f_distal/pst/f_d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 scale=0.001 0.001 0.001; visual mesh filename=package://sr_description/meshes/components/f_distal/pst/f_d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 scale=0.001 0.001 0.001
- link rh_mfknuckle: geometry collision cylinder length=0.014 radius=0.007; visual mesh filename=package://sr_description/meshes/components/f_knuckle/f_knuc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 scale=0.001 0.001 0.001
- link rh_mfmiddle: geometry collision cylinder length=0.025 radius=0.007; collision sphere radius=0.007
- link rh_mfproximal: geometry collision cylinder length=0.040 radius=0.007; visual mesh filename=package://sr_description/meshes/components/f_proximal/f_pro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 scale=0.001 0.001 0.001
- link rh_palm: geometry collision box size=0.018 0.024 0.004; collision box size=0.020 0.024 0.040
- link rh_rfdistal: geometry collision mesh filename=package://sr_description/meshes/components/f_distal/pst/f_d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 scale=0.001 0.001 0.001; visual mesh filename=package://sr_description/meshes/components/f_distal/pst/f_d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 scale=0.001 0.001 0.001
- link rh_rfknuckle: geometry collision cylinder length=0.014 radius=0.007; visual mesh filename=package://sr_description/meshes/components/f_knuckle/f_knuc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 scale=0.001 0.001 0.001
- link rh_rfmiddle: geometry collision cylinder length=0.025 radius=0.007; collision sphere radius=0.007
- link rh_rfproximal: geometry collision cylinder length=0.040 radius=0.007; visual mesh filename=package://sr_description/meshes/components/f_proximal/f_pro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 scale=0.001 0.001 0.001
- link rh_thdistal: geometry collision mesh filename=package://sr_description/meshes/components/th_distal/pst/th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 scale=0.001 0.001 0.001; visual mesh filename=package://sr_description/meshes/components/th_distal/pst/th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 scale=0.001 0.001 0.001
- link rh_thmiddle: geometry collision cylinder length=0.014 radius=0.010; collision cylinder length=0.018 radius=0.011
- link rh_thproximal: geometry collision cylinder length=0.018 radius=0.012; visual mesh filename=package://sr_description/meshes/components/th_proximal/th_p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 scale=0.001 0.001 0.001
Joints:
- removed joint rh_base_joint
- removed joint virtual_px_joint
- removed joint virtual_py_joint
- removed joint virtual_pz_joint
- removed joint virtual_rp_joint
- removed joint virtual_rr_joint
- removed joint virtual_ry_joint
- added joint rh_WRJ1: type revolute, parent rh_wrist, child rh_palm, origin xyz=0 0 0.034 rpy=0 0 0, axis 1 0 0, limit lower=-0.6981317007977318 upper=0.4886921905584123 effort=30 velocity=2.0
- added joint rh_WRJ2: type revolute, parent rh_forearm, child rh_wrist, origin xyz=0 -0.010 0.21301 rpy=0 0 0, axis 0 1 0, limit lower=-0.5235987755982988 upper=0.17453292519943295 effort=10 velocity=2.0
- added joint rh_ee_fixed_joint: type fixed, parent rh_palm, child rh_manipulator, origin xyz=0.0 0.0 0.05 rpy=0.0 0.0 0.0
- added joint rh_world_joint: type fixed, parent world, child rh_forearm, origin xyz=0.0 0.0 0.0 rpy=0.0 0.0 0.0
- joint rh_FFJ1: limit lower=0 upper=1.57079632679 effort=2 velocity=2.0 -> lower=0 upper=1.5707963267948966 effort=2 velocity=2.0
- joint rh_FFJ2: limit lower=0 upper=1.57079632679 effort=2 velocity=2.0 -> lower=0 upper=1.5707963267948966 effort=2 velocity=2.0
- joint rh_FFJ3: limit lower=0 upper=1.57079632679 effort=2 velocity=2.0 -> lower=-0.2617993877991494 upper=1.5707963267948966 effort=2 velocity=2.0
- joint rh_FFJ4: axis 0 -1.0 0 -> 0 -1 0; limit lower=-0.349065850399 upper=0.349065850399 effort=2 velocity=2.0 -> lower=-0.3490658503988659 upper=0.3490658503988659 effort=2 velocity=2.0
- joint rh_LFJ1: limit lower=0 upper=1.57079632679 effort=2 velocity=2.0 -> lower=0 upper=1.5707963267948966 effort=2 velocity=2.0
- joint rh_LFJ2: limit lower=0 upper=1.57079632679 effort=2 velocity=2.0 -> lower=0 upper=1.5707963267948966 effort=2 velocity=2.0
- joint rh_LFJ3: limit lower=0 upper=1.57079632679 effort=2 velocity=2.0 -> lower=-0.2617993877991494 upper=1.5707963267948966 effort=2 velocity=2.0
- joint rh_LFJ4: axis 0 1.0 0 -> 0 1 0; limit lower=-0.349065850399 upper=0.349065850399 effort=2 velocity=2.0 -> lower=-0.3490658503988659 upper=0.3490658503988659 effort=2 velocity=2.0; origin xyz=0 0 0.06579 rpy=0 0 0 -> xyz=0.05397275 0 0.03779463 rpy=0 0.9599 0
- joint rh_LFJ5: axis 0.573576436 0 0.819152044 -> 1 0 0; limit lower=0 upper=0.785398163397 effort=2 velocity=2.0 -> lower=0 upper=0.7853981633974483 effort=2 velocity=2.0; origin xyz=-0.033 0 0.02071 rpy=0 0 0 -> xyz=-0.033 0 0.02071 rpy=0 -0.9599 0
- joint rh_MFJ1: limit lower=0 upper=1.57079632679 effort=2 velocity=2.0 -> lower=0 upper=1.5707963267948966 effort=2 velocity=2.0
- joint rh_MFJ2: limit lower=0 upper=1.57079632679 effort=2 velocity=2.0 -> lower=0 upper=1.5707963267948966 effort=2 velocity=2.0
- joint rh_MFJ3: limit lower=0 upper=1.57079632679 effort=2 velocity=2.0 -> lower=-0.2617993877991494 upper=1.5707963267948966 effort=2 velocity=2.0
- joint rh_MFJ4: axis 0 -1.0 0 -> 0 -1 0; limit lower=-0.349065850399 upper=0.349065850399 effort=2 velocity=2.0 -> lower=-0.3490658503988659 upper=0.3490658503988659 effort=2 velocity=2.0
- joint rh_RFJ1: limit lower=0 upper=1.57079632679 effort=2 velocity=2.0 -> lower=0 upper=1.5707963267948966 effort=2 velocity=2.0
- joint rh_RFJ2: limit lower=0 upper=1.57079632679 effort=2 velocity=2.0 -> lower=0 upper=1.5707963267948966 effort=2 velocity=2.0
- joint rh_RFJ3: limit lower=0 upper=1.57079632679 effort=2 velocity=2.0 -> lower=-0.2617993877991494 upper=1.5707963267948966 effort=2 velocity=2.0
- joint rh_RFJ4: axis 0 1.0 0 -> 0 1 0; limit lower=-0.349065850399 upper=0.349065850399 effort=2 velocity=2.0 -> lower=-0.3490658503988659 upper=0.3490658503988659 effort=2 velocity=2.0
- joint rh_THJ1: limit lower=0 upper=1.57079632679 effort=1.0 velocity=4.0 -> lower=-0.2617993877991494 upper=1.5707963267948966 effort=1.0 velocity=4.0; origin xyz=0 0 0.032 rpy=0 0 -1.57079632679 -> xyz=0 0 0.032 rpy=0 0 0
- joint rh_THJ2: axis 0 -1 0 -> 1 0 0; limit lower=-0.698131700798 upper=0.698131700798 effort=2.0 velocity=2.0 -> lower=-0.6981317007977318 upper=0.6981317007977318 effort=2.0 velocity=2.0
- joint rh_THJ3: axis 1 0 0 -> 0 1 0; limit lower=-0.209439510239 upper=0.209439510239 effort=2.0 velocity=4.0 -> lower=-0.20943951023931953 upper=0.20943951023931953 effort=2.0 velocity=4.0
- joint rh_THJ4: axis 1.0 0 0 -> 0 1 0; limit lower=0.0 upper=1.2217304764 effort=3 velocity=4.0 -> lower=0.0 upper=1.2217304763960306 effort=3 velocity=4.0
- joint rh_THJ5: axis 0 0 -1.0 -> 0 0 -1; limit lower=-1.0471975512 upper=1.0471975512 effort=5.0 velocity=4.0 -> lower=-1.0471975511965976 upper=1.0471975511965976 effort=5.0 velocity=4.0; origin xyz=0.034 -0.0085 0.029 rpy=0 0.785398163397 0.0 -> xyz=0.034 -0.00858 0.029 rpy=-0.7853981633974483 0 -1.5707963267948966
